File: KiCad_Project/usb-pd-15v-3a.kicad_sch (KiCad schematic)
At the start: 0 parts

Commit message: update psu git
Parts:
- added C1: 47n, Capacitor_SMD:C_0603_1608Metric, symbol Device:C_Small
- added C10, C11, C2, C3, C4, C6, C7, C8, C9: 100nF, Capacitor_SMD:C_0805_2012Metric, symbol Device:C_Small
- added C12, C5: 22n, Capacitor_SMD:C_0603_1608Metric, symbol Device:C_Small
- added C_in1, C_in3: 220uF, Capacitor_SMD:CP_Elec_10x7.7, symbol Device:C_Polarized_Small
- added C_in2, C_in4, C_in6: 100nF, Capacitor_SMD:C_1206_3216Metric, symbol Device:C_Small
- added C_in5: 100uF, Capacitor_SMD:CP_Elec_6.3x7.7, symbol Device:C_Polarized_Small
- added C_out1, C_out2, C_out3: 47u, Capacitor_SMD:C_1206_3216Metric, symbol Device:C_Small
- added C_out4, C_out5, C_out6, C_out7, C_out8, C_out9: 100uF, Inductor_SMD:L_1210_3225Metric, symbol Device:C_Small
- added D1, D5, D6: SS54, Diode_SMD:D_SMA, symbol Device:D_Schottky
- added D2, D3, D4: (no value), LED_THT:LED_D3.0mm, symbol Device:LED_Small
- added H1, H2: MountingHole_Pad, MountingHole:MountingHole_3.2mm_M3_Pad_TopOnly, symbol Mechanical:MountingHole_Pad
- added J1: 2.5mm/5.5mm (PC-G2.5-PCB), Connectors:DC_Barrel_Jack_2.5mm_5.7mm_Verrtical, symbol Connector:Barrel_Jack_Switch
- added J2: Conn_02x08_Odd_Even, Connector_IDC:IDC-Header_2x08_P2.54mm_Vertical, symbol Connector_Generic:Conn_02x08_Odd_Even
- added L1, L2, L3: 33uH, Inductor_SMD:L_12x12mm_H8mm, symbol Device:L
- added R1, R15, R8: 1k2, Resistor_SMD:R_0805_2012Metric_Pad1.20x1.40mm_HandSolder, symbol Device:R
- added R10, R11, R12, R13, R3, R4: 47k, Resistor_SMD:R_0603_1608Metric, symbol Device:R
- added R14, R9: 15k, Resistor_SMD:R_0805_2012Metric_Pad1.20x1.40mm_HandSolder, symbol Device:R
- added R2: 6k2, Resistor_SMD:R_0805_2012Metric_Pad1.20x1.40mm_HandSolder, symbol Device:R
- added R5: 2k2, Resistor_SMD:R_0603_1608Metric, symbol Device:R
- added R6, R7: 8k2, Resistor_SMD:R_0603_1608Metric, symbol Device:R
- added U1, U3, U6: LM2596S-ADJ, Package_TO_SOT_SMD:TO-263-5_TabPin3, symbol Regulator_Switching:LM2596S-ADJ
- added U2: L7805, Package_TO_SOT_SMD:TO-263-3_TabPin2, symbol Regulator_Linear:L7805
- added U4: L7812, Package_TO_SOT_SMD:TO-263-3_TabPin2, symbol Regulator_Linear:L7812
- added U5: L7912, Package_TO_SOT_SMD:TO-263-3_TabPin2, symbol Regulator_Linear:L7912
Connections:
- new net: C1.2, R1.1, R2.1, U1.4 (FB)
- new net: C12.2, R14.2, R15.1, U6.4 (FB)
- new net: C5.1, C7.2, C_out4.2, C_out5.1, L2.2, R9.1, U4.1 (IN)
- new net: C5.2, R8.1, R9.2, U3.4 (FB)
- new net: C2.2, R3.1
- new net: R3.2, R4.1, U1.5 (~{ON}/OFF)
- new net: D3.2 (A), R6.2
- new net: C11.2, R13.1
- new net: R12.1, R13.2, U6.5 (~{ON}/OFF)
- new net: C1.1, C3.2, C_out1.2, C_out2.1, L1.2, R2.2, U2.1 (IN)
- new net: C6.2, R10.1
- new net: D6.1 (K), L3.2, U6.2 (OUT)
- new net: D5.1 (K), L2.1, U3.2 (OUT)
- new net: R10.2, R11.1, U3.5 (~{ON}/OFF)
- new net: D1.1 (K), L1.1, U1.2 (OUT)
- new net: D2.2 (A), R5.2
- new net: D4.2 (A), R7.2
- new net +12V: C8.1, C_out6.1, J2.10 (Pin_10), J2.9 (Pin_9), R6.1, U4.3 (OUT)
- new net +5V: C4.1, C_out3.1, J2.11 (Pin_11), J2.12 (Pin_12), R5.1, U2.3 (OUT)
- new net -12V: C10.2, C_out9.2, D4.1 (K), J2.1 (Pin_1), J2.2 (Pin_2), U5.3 (VO)
- new net -14.5V: C9.1, C_in5.2, C_in6.1, C_out7.1, C_out8.2, D6.2 (A), R12.2, R15.2, U5.2 (VI), U6.3 (GND)
- new net GND: C10.1, C12.1, C3.1, C4.2, C7.1, C8.2, C9.2, C_in1.2, C_in2.2, C_in3.2, C_in4.2, C_out1.1, C_out2.2, C_out3.2, C_out4.1, C_out5.2, C_out6.2, C_out7.2, C_out8.1, C_out9.1, D1.2 (A), D2.1 (K), D3.1 (K), D5.2 (A), H1.1, H2.1, J1.1, J2.3 (Pin_3), J2.4 (Pin_4), J2.5 (Pin_5), J2.6 (Pin_6), J2.7 (Pin_7), J2.8 (Pin_8), L3.1, R1.2, R11.2, R14.1, R4.2, R7.1, R8.2, U1.3 (GND), U2.2 (GND), U3.3 (GND), U4.2 (GND), U5.1 (GND)
- new net Vin: C11.1, C2.1, C6.1, C_in1.1, C_in2.1, C_in3.1, C_in4.1, C_in5.1, C_in6.2, J1.2, U1.1 (VIN), U3.1 (VIN), U6.1 (VIN)
- no-connect marks 0 -> 5
Other:
- removed sheet interface
- removed sheet main_psu
- note added: "15V - 20V DC input"
- note added: "Eurorack Output"
- note added: "LDO to +12V"
- note added: "LDO to +5V"
- note added: "LDO to -12V"
- note added: "Power Leds"
- note added: "Step Down to +14.5V"
- note added: "Step Down to +7.5V"
- note added: "Step Down to -14.5V"
- company: (none) -> GSS
- title: (none) -> PSU for Eurorack
